Commit message: Add files via upload

File: uvone_robot_description/urdf/include/astra.urdf.xacro (robot description, xacro)
@@ -41,5 +41,5 @@
     <xacro:macro name="sensor_astra" params="parent posz">
         <joint name="camera_rgb_joint" type="fixed">
-        <origin xyz="0.012 -0.070 ${posz}"
+        <origin xyz="0.012 0.010 ${posz}"
                 rpy="0 0.37 0"/>
         <parent link="${parent}"/>
@@ -48,5 +48,5 @@
         <link name="camera_rgb_frame"/>
         <joint name="camera_rgb_optical_joint" type="fixed">
-        <origin xyz="0 -0.014 0" rpy="${-M_PI/2} 0 ${-M_PI/2}" />
+        <origin xyz="0 0 0" rpy="${-M_PI/2} 0 ${-M_PI/2}" />
         <parent link="camera_rgb_frame" />
         <child link="camera_rgb_optical_frame" />
@@ -54,5 +54,5 @@
         <link name="camera_rgb_optical_frame"/>
         <joint name="camera_depth_joint" type="fixed">
-        <origin xyz="0 -0.036 0" rpy="0 0 0" /><!-- ha cambiado !! posy-->
+        <origin xyz="0 -0.016 0" rpy="0 0 0" /><!-- ha cambiado !! posy-->
         <parent link="camera_rgb_frame" />
         <child link="camera_depth_frame" />

File: uvone_robot_description/urdf/model.urdf.xacro (robot description, xacro)
@@ -33,4 +33,4 @@
   </link>
   <!-- Camara astra -->
-  <xacro:sensor_astra parent="base_link" posz="1.238"/>  <!-- Primer escalon: posz=0.718 --> <!-- Segundo escalon: posz=1.358 -->
+  <xacro:sensor_astra parent="base_link" posz="1.358"/>  <!-- Primer escalon: posz=0.718 --> <!-- Segundo escalon: posz=1.358 -->
 </robot>

Commit message: Add files via upload

File: uvone_robot_description/urdf/include/astra.urdf.xacro (robot description, xacro)
@@ -41,10 +41,20 @@
     <xacro:macro name="sensor_astra" params="parent posz">
         <joint name="camera_rgb_joint" type="fixed">
-        <origin xyz="0.012 0.010 ${posz}"
-                rpy="0 0.37 0"/>
+        <origin xyz="0.1 0 ${posz}"
+                rpy="0 0 0"/>
         <parent link="${parent}"/>
         <child link="camera_rgb_frame" />
         </joint>
-        <link name="camera_rgb_frame"/>
+        <link name="camera_rgb_frame">
+    <visual>
+      <geometry>
+        <mesh filename="package://uvone_robot_description/meshes/astra.dae" scale="0.75 0.75 0.75"/>
+      </geometry>
+      <origin rpy="1.57 0 1.57" xyz="0 0 -0.1" />
+      <material name="black">
+        <color rgba="0.2 0.2 0.2 1" />
+      </material>
+    </visual>
+  </link>
         <joint name="camera_rgb_optical_joint" type="fixed">
         <origin xyz="0 0 0" rpy="${-M_PI/2} 0 ${-M_PI/2}" />

File: uvone_robot_description/urdf/mopad.urdf.xacro (robot description, xacro)
@@ -16,5 +16,5 @@
 <!-- RPlidar -->
   <joint name="rplidar_joint" type="fixed">
-    <origin rpy="0 0 -3.1415926536" xyz="0.110 0 0.108" />
+    <origin rpy="3.1415926536 0 3.1415926536" xyz="0.110 0.0 0.108" />
     <parent link="base_link"/>
     <child link="rplidar"/>
@@ -25,5 +25,5 @@
         <mesh filename="package://uvone_robot_description/meshes/rplidar.stl" scale="0.001 0.001 0.001"/>
       </geometry>
-      <origin rpy="-1.57 0 0" xyz="0 -0.07 0.04" />
+      <origin rpy="1.57 0 0" xyz="0 0.075 -0.04" />
       <material name="black">
         <color rgba="0.2 0.2 0.2 1" />
@@ -32,21 +32,21 @@
   </link>
   <xacro:rplidar_sim/>
- <!-- Camara astra  -->
-  <joint name="astra_joint" type="fixed">
-    <origin rpy="1.57 0 1.57" xyz="0.10 0 0.29" />
+ <!-- Camara astra (Esta parte no vale) -->
+   <!--<joint name="astra_joint" type="fixed">
+    <origin rpy="0 0 0" xyz="0.10 0 0.29" />
     <parent link="base_link"/>
     <child link="astra"/>
   </joint>
-  <link name="astra">
+ <link name="astra">
     <visual>
       <geometry>
         <mesh filename="package://uvone_robot_description/meshes/astra.dae" scale="0.75 0.75 0.75"/>
       </geometry>
-      <origin rpy="0 0 0" xyz="0 0 0" />
+      <origin rpy="1.57 0 1.57" xyz="0 0 0" />
       <material name="black">
         <color rgba="0.2 0.2 0.2 1" />
       </material>
     </visual>
-  </link>
-  <xacro:sensor_astra parent="base_link" posz="0.3" />
+  </link> -->
+  <xacro:sensor_astra parent="base_link" posz="0.4" />
 </robot>
