Commit message: Finalizado el modelo

File: mopad_description/urdf/include/astra.urdf.xacro (robot description, xacro)
@@ -1,4 +1,4 @@
 <?xml version="1.0"?>
-<robot name="rplidar_sim" xmlns:xacro="http://ros.org/wiki/xacro">
+<robot name="astra_sensor" xmlns:xacro="http://ros.org/wiki/xacro">
   <xacro:macro name="sim_3dsensor">
     <gazebo reference="camera_rgb_frame">
@@ -48,9 +48,9 @@
 	<!-- .........................................................-->
         <link name="camera_rgb_frame">
-    <visual>
+ <visual>
       <geometry>
-        <mesh filename="package://mopad_description/meshes/astra.dae" scale="0.75 0.75 0.75"/>
+        <mesh filename="package://uvone_robot_description/meshes/astra.stl" scale="0.001 0.001 0.001"/>
       </geometry>
-      <origin rpy="1.57 0 1.57" xyz="0 0 0" />
+      <origin rpy="1.62 0 1.57" xyz="0.05 0.025 0.039" />
       <material name="black">
         <color rgba="0.2 0.2 0.2 1" />
@@ -77,22 +77,4 @@
         </joint>
         <link name="camera_depth_optical_frame"/>
-	<!-- .........................................................-->
-	<joint name="camera_joint" type="fixed">
-     	 <origin xyz="0 0 0" rpy="0 0 0"/>
-      	<parent link="camera_rgb_frame"/>
-      	<child link="camera_link"/>
-    	</joint>
-    	<link name="camera_link">
-	   <visual>
-      		<geometry>
-        	<mesh filename="package://mopad_description/meshes/astra.dae" 			scale="0.75 0.75 0.75"/>
-      		</geometry>
-      		<origin rpy="1.57 0 1.57" xyz="0 0 0" />
-      		<material name="black">
-      		  <color rgba="0.2 0.2 0.2 1" />
-      		</material>
-           </visual>
- 	 </link>
-	<!-- .........................................................-->
         <!-- RGBD sensor for simulation, same as Kinect -->
         <xacro:sim_3dsensor/>

File: mopad_description/urdf/mopad.urdf.xacro (robot description, xacro)
@@ -7,9 +7,9 @@
 -->
 <robot name="mopad" xmlns:xacro="http://ros.org/wiki/xacro">
- <!-- <xacro:include filename="$(find turtlebot_description)/urdf/turtlebot_common_library.urdf.xacro" />   -->
+  <xacro:include filename="$(find turtlebot_description)/urdf/turtlebot_common_library.urdf.xacro" />
   <xacro:include filename="$(find kobuki_description)/urdf/kobuki.urdf.xacro" />
-  <xacro:include filename="$(find mopad_description)/urdf/include/hexagons.urdf.xacro"/>
-  <xacro:include filename="$(find mopad_description)/urdf/include/rplidar.urdf.xacro" />
-  <xacro:include filename="$(find mopad_description)/urdf/include/astra.urdf.xacro" />
+  <xacro:include filename="$(find uvone_robot_description)/urdf/include/hexagons.urdf.xacro"/>
+  <xacro:include filename="$(find uvone_robot_description)/urdf/include/rplidar.urdf.xacro" />
+  <xacro:include filename="$(find uvone_robot_description)/urdf/include/astra.urdf.xacro" />
   <xacro:kobuki/>
   <xacro:stack_hexagons parent="base_link"/>
@@ -23,5 +23,5 @@
     <visual>
       <geometry>
-        <mesh filename="package://mopad_description/meshes/rplidar.stl" scale="0.001 0.001 0.001"/>
+        <mesh filename="package://uvone_robot_description/meshes/rplidar.stl" scale="0.001 0.001 0.001"/>
       </geometry>
       <origin rpy="1.57 0 0" xyz="0 0.075 -0.04" />
@@ -32,21 +32,4 @@
   </link>
   <xacro:rplidar_sim/>
- <!-- Camara astra (Esta parte no vale)
-    <joint name="astra_joint" type="fixed">
-    <origin rpy="0 0 0" xyz="0.10 0 0.29" />
-    <parent link="base_link"/>
-    <child link="astra"/>
-  </joint>
- <link name="astra">
-    <visual>
-      <geometry>
-        <mesh filename="package://mopad_description/meshes/astra.dae" scale="0.75 0.75 0.75"/>
-      </geometry>
-      <origin rpy="1.57 0 1.57" xyz="0 0 0" />
-      <material name="black">
-        <color rgba="0.2 0.2 0.2 1" />
-      </material>
-    </visual>
-  </link> -->
-   <xacro:sensor_astra parent="base_link" posz="0.32"/>
+   <xacro:sensor_astra parent="base_link" posz="0.31"/>
 </robot>

Commit message: Add files via upload

File: mopad_description/urdf/include/astra.urdf.xacro (robot description, xacro)
@@ -47,16 +47,15 @@
         </joint>
 	<!-- .........................................................-->
-        <link name="camera_rgb_frame">
- <visual>
-      <geometry>
-        <mesh filename="package://uvone_robot_description/meshes/astra.stl" scale="0.001 0.001 0.001"/>
-      </geometry>
-      <origin rpy="1.62 0 1.57" xyz="0.05 0.025 0.039" />
-      <material name="black">
-        <color rgba="0.2 0.2 0.2 1" />
-      </material>
-    </visual>
+        <link name="camera_rgb_frame" >
+ 	<visual>
+      	<geometry>
+      		  <mesh filename="package://mopad_description/meshes/astra.stl" scale="0.001 0.001 0.001"/>
+      	</geometry>
+      	<origin rpy="1.62 0 1.57" xyz="0.05 0.025 0.039" />
+      	<material name="black">
+        	<color rgba="0.2 0.2 0.2 1" />
+      	</material>
+   	 </visual>
   </link>
-	<!-- .........................................................-->
         <joint name="camera_rgb_optical_joint" type="fixed">
         <origin xyz="0 0 0" rpy="${-M_PI/2} 0 ${-M_PI/2}" />

File: mopad_description/urdf/include/hexagons.urdf.xacro (robot description, xacro)
@@ -162,5 +162,5 @@
      <xacro:stack_3d_sensor_pole parent="${parent}" number="0" x_loc= "0.11" y_loc= "0.1" z_loc="0.235"/>
     <xacro:stack_3d_sensor_pole parent="${parent}" number="1" x_loc= "0.11" y_loc="-0.1" z_loc="0.235"/>
-<!-- <joint name="plate_camera_joint" type="fixed">
+ <joint name="plate_camera_joint" type="fixed">
       <origin xyz="0.122 0.0 0.27" rpy="0 0 1.57"/>
       <parent link="${parent}"/>
@@ -173,6 +173,9 @@
          <mesh filename="package://mopad_description/meshes/pieza.stl" scale="0.00102 0.0012 0.0012"/>
         </geometry>
+	<material name="black">
+        	<color rgba="0.2 0.2 0.2 1" />
+      	</material>
       </visual>
-    </link> -->
+    </link>
   </xacro:macro>
 </robot>

File: mopad_description/urdf/mopad.urdf.xacro (robot description, xacro)
@@ -9,7 +9,7 @@
   <xacro:include filename="$(find turtlebot_description)/urdf/turtlebot_common_library.urdf.xacro" />
   <xacro:include filename="$(find kobuki_description)/urdf/kobuki.urdf.xacro" />
-  <xacro:include filename="$(find uvone_robot_description)/urdf/include/hexagons.urdf.xacro"/>
-  <xacro:include filename="$(find uvone_robot_description)/urdf/include/rplidar.urdf.xacro" />
-  <xacro:include filename="$(find uvone_robot_description)/urdf/include/astra.urdf.xacro" />
+  <xacro:include filename="$(find mopad_description)/urdf/include/hexagons.urdf.xacro"/>
+  <xacro:include filename="$(find mopad_description)/urdf/include/rplidar.urdf.xacro" />
+  <xacro:include filename="$(find mopad_description)/urdf/include/astra.urdf.xacro" />
   <xacro:kobuki/>
   <xacro:stack_hexagons parent="base_link"/>
@@ -23,5 +23,5 @@
     <visual>
       <geometry>
-        <mesh filename="package://uvone_robot_description/meshes/rplidar.stl" scale="0.001 0.001 0.001"/>
+        <mesh filename="package://mopad_description/meshes/rplidar.stl" scale="0.001 0.001 0.001"/>
       </geometry>
       <origin rpy="1.57 0 0" xyz="0 0.075 -0.04" />
